Commit message: Start controller with namespaces (#15)
* Configure xacro via launch args

Signed-off-by: Yadunund <yadunund@gmail.com>

* Namespace controllers

Signed-off-by: Yadunund <yadunund@gmail.com>

* Allow robot links and joints to be namespaced

Signed-off-by: Yadunund <yadunund@gmail.com>

* Pass ros2_control.xacro and controller_config files as launch args

Signed-off-by: Yadunund <yadunund@gmail.com>

* Pre-commit

---------

Signed-off-by: Yadunund <yadunund@gmail.com>
Co-authored-by: JafarAbdi <jafar.uruc@gmail.com>

File: so_arm100_description/control/so_arm100.ros2_control.xacro (robot description, xacro)
@@ -1,5 +1,8 @@
 <?xml version="1.0" ?>
 <robot xmlns:xacro="http://www.ros.org/wiki/xacro">
-  <xacro:macro name="ros2_control" params="ros2_control_hardware_type">
+  <xacro:macro
+    name="ros2_control"
+    params="prefix ros2_control_hardware_type usb_port"
+  >
     <ros2_control name="SO-ARM100" type="system">
       <hardware>
@@ -9,8 +12,8 @@
         <xacro:if value="${ros2_control_hardware_type == 'real'}">
           <plugin>feetech_ros2_driver/FeetechHardwareInterface</plugin>
-          <param name="usb_port">/dev/LeRobotFollower</param>
+          <param name="usb_port">${usb_port}</param>
         </xacro:if>
       </hardware>
-      <joint name="shoulder_pan_joint">
+      <joint name="${prefix}shoulder_pan_joint">
         <param name="initial_position">0.0</param>
         <param name="id">1</param>
@@ -21,5 +24,5 @@
         <state_interface name="velocity" />
       </joint>
-      <joint name="shoulder_lift_joint">
+      <joint name="${prefix}shoulder_lift_joint">
         <param name="id">2</param>
         <param name="p_cofficient">16</param>
@@ -30,5 +33,5 @@
         <state_interface name="velocity" />
       </joint>
-      <joint name="elbow_joint">
+      <joint name="${prefix}elbow_joint">
         <param name="id">3</param>
         <param name="offset">2080</param>
@@ -39,5 +42,5 @@
         <state_interface name="velocity" />
       </joint>
-      <joint name="wrist_pitch_joint">
+      <joint name="${prefix}wrist_pitch_joint">
         <param name="id">4</param>
         <param name="offset">3110</param>
@@ -48,5 +51,5 @@
         <state_interface name="velocity" />
       </joint>
-      <joint name="wrist_roll_joint">
+      <joint name="${prefix}wrist_roll_joint">
         <param name="id">5</param>
         <param name="offset">1024</param>
@@ -57,5 +60,5 @@
         <state_interface name="velocity" />
       </joint>
-      <joint name="jaw_joint">
+      <joint name="${prefix}jaw_joint">
         <param name="id">6</param>
         <param name="offset">2070</param>

File: so_arm100_description/urdf/so_arm100.urdf.xacro (robot description, xacro)
@@ -2,10 +2,23 @@
 <robot xmlns:xacro="http://www.ros.org/wiki/xacro" name="so_100arm">
   <xacro:arg name="ros2_control_hardware_type" default="mock_components" />
-  <xacro:include filename="so_arm100.urdf" />
-  <xacro:include
-    filename="$(find so_arm100_description)/control/so_arm100.ros2_control.xacro"
+  <xacro:arg
+    name="ros2_control_file"
+    default="$(find so_arm100_description)/control/so_arm100.ros2_control.xacro"
   />
+  <xacro:arg
+    name="urdf_file"
+    default="$(find so_arm100_description)/urdf/so_arm100_macro.xacro"
+  />
+  <xacro:arg name="usb_port" default="/dev/LeRobotFollower" />
+  <xacro:arg name="prefix" default="" />
+  <!-- Robot description -->
+  <xacro:include filename="$(arg urdf_file)" />
+  <xacro:so_arm100 prefix="$(arg prefix)" />
+  <!-- ros2_control description -->
+  <xacro:include filename="$(arg ros2_control_file)" />
   <xacro:ros2_control
+    prefix="$(arg prefix)"
     ros2_control_hardware_type="$(arg ros2_control_hardware_type)"
+    usb_port="$(arg usb_port)"
   />
 </robot>

Commit message: enabling so101. check in anyway (although it doesn't work yet) before exploring other approach

File: so_arm100_description/control/so_arm100.ros2_control.xacro (robot description, xacro)
@@ -23,4 +23,8 @@
         <state_interface name="position" />
         <state_interface name="velocity" />
+        <param name="min_position">-1.91986</param>
+        <param name="max_position">1.91986</param>
+        <param name="max_velocity">10.0</param>
+        <param name="max_effort">10.0</param>
       </joint>
       <joint name="${prefix}shoulder_lift_joint">
@@ -32,4 +36,8 @@
         <state_interface name="position" />
         <state_interface name="velocity" />
+        <param name="min_position">-1.74533</param>
+        <param name="max_position">1.74533</param>
+        <param name="max_velocity">10.0</param>
+        <param name="max_effort">10.0</param>
       </joint>
       <joint name="${prefix}elbow_joint">
@@ -41,4 +49,8 @@
         <state_interface name="position" />
         <state_interface name="velocity" />
+        <param name="min_position">-1.69</param>
+        <param name="max_position">1.69</param>
+        <param name="max_velocity">10.0</param>
+        <param name="max_effort">10.0</param>
       </joint>
       <joint name="${prefix}wrist_pitch_joint">
@@ -50,4 +62,8 @@
         <state_interface name="position" />
         <state_interface name="velocity" />
+        <param name="min_position">-1.65806</param>
+        <param name="max_position">1.65806</param>
+        <param name="max_velocity">10.0</param>
+        <param name="max_effort">10.0</param>
       </joint>
       <joint name="${prefix}wrist_roll_joint">
@@ -59,4 +75,8 @@
         <state_interface name="position" />
         <state_interface name="velocity" />
+        <param name="min_position">-2.74385</param>
+        <param name="max_position">2.84121</param>
+        <param name="max_velocity">10.0</param>
+        <param name="max_effort">10.0</param>
       </joint>
       <joint name="${prefix}jaw_joint">
@@ -68,4 +88,8 @@
         <state_interface name="position" />
         <state_interface name="velocity" />
+        <param name="min_position">-0.174533</param>
+        <param name="max_position">1.74533</param>
+        <param name="max_velocity">10.0</param>
+        <param name="max_effort">10.0</param>
       </joint>
     </ros2_control>

File: so_arm100_description/urdf/so_arm100_macro.xacro (robot description, xacro)
@@ -42,5 +42,5 @@
         <origin xyz="0 0 0" rpy="0 0 0" />
         <geometry>
-          <mesh filename="package://so_arm100_description/meshes/Base.STL" />
+          <mesh filename="package://so_arm100_description/SO-ARM101-Assets/base_motor_holder_so101_v1.stl" />
         </geometry>
         <material name="">
@@ -53,5 +53,5 @@
         <origin xyz="0 0 0" rpy="0 0 0" />
         <geometry>
-          <mesh filename="package://so_arm100_description/meshes/Base.STL" />
+          <mesh filename="package://so_arm100_description/SO-ARM101-Assets/base_motor_holder_so101_v1.stl" />
         </geometry>
       </collision>
@@ -74,31 +74,36 @@
       </inertial>
       <visual>
-        <origin xyz="0 0 0" rpy="0 0 0" />
-        <geometry>
-          <mesh
-            filename="package://so_arm100_description/meshes/Rotation_Pitch.STL"
-          />
-        </geometry>
-        <material name="">
-          <color
-            rgba="0.792156862745098 0.819607843137255 0.933333333333333 1"
-          />
-        </material>
-      </visual>
-      <collision>
-        <origin xyz="0 0 0" rpy="0 0 0" />
-        <geometry>
-          <mesh
-            filename="package://so_arm100_description/meshes/Rotation_Pitch.STL"
-          />
+        <origin xyz="-0.0303992 0.000422241 -0.0417" rpy="1.5708 1.5708 0" />
+        <geometry>
+          <mesh filename="package://so_arm100_description/SO-ARM101-Assets/sts3215_03a_v1.stl" />
+        </geometry>
+        <material name="sts3215"/>
+      </visual>
+      <visual>
+        <origin xyz="-0.0675992 -0.000177759 0.0158499" rpy="1.5708 -1.5708 0" />
+        <geometry>
+          <mesh filename="package://so_arm100_description/SO-ARM101-Assets/motor_holder_so101_base_v1.stl" />
+        </geometry>
+        <material name="3d_printed"/>
+      </visual>
+      <visual>
+        <origin xyz="0 0 0" rpy="0 0 0" />
+        <geometry>
+          <mesh filename="package://so_arm100_description/SO-ARM101-Assets/rotation_pitch_so101_v1.stl" />
+        </geometry>
+      </visual>
+      <collision>
+        <origin xyz="-0.0303992 0.000422241 -0.0417" rpy="1.5708 1.5708 0" />
+        <geometry>
+          <mesh filename="package://so_arm100_description/SO-ARM101-Assets/sts3215_03a_v1.stl" />
         </geometry>
       </collision>
     </link>
     <joint name="${prefix}shoulder_pan_joint" type="revolute">
-      <origin xyz="0 -0.0452 0.0165" rpy="1.5708 0 0" />
+      <origin xyz="0.0388353 0 0.0459" rpy="0 0 0" />
       <parent link="${prefix}base" />
       <child link="${prefix}shoulder_link" />
-      <axis xyz="0 -1 0" />
-      <limit lower="-2.0" upper="2.0" effort="1" velocity="1" />
+      <axis xyz="0 0 1" />
+      <limit effort="10" velocity="10" lower="-1.91986" upper="1.91986" />
     </joint>
     <link name="${prefix}upper_arm_link">
@@ -121,29 +126,27 @@
         <origin xyz="0 0 0" rpy="0 0 0" />
         <geometry>
-          <mesh
-            filename="package://so_arm100_description/meshes/Upper_Arm.STL"
-          />
-        </geometry>
-        <material name="">
-          <color
-            rgba="0.792156862745098 0.819607843137255 0.933333333333333 1"
-          />
-        </material>
-      </visual>
-      <collision>
-        <origin xyz="0 0 0" rpy="0 0 0" />
-        <geometry>
-          <mesh
-            filename="package://so_arm100_description/meshes/Upper_Arm.STL"
-          />
+          <mesh filename="package://so_arm100_description/SO-ARM101-Assets/sts3215_03a_v1.stl" />
+        </geometry>
+        <material name="sts3215"/>
+      </visual>
+      <visual>
+        <origin xyz="0 0 0" rpy="0 0 0" />
+        <geometry>
+          <mesh filename="package://so_arm100_description/SO-ARM101-Assets/upper_arm_so101_v1.stl" />
+        </geometry>
+      </visual>
+      <collision>
+        <origin xyz="0 0 0" rpy="0 0 0" />
+        <geometry>
+          <mesh filename="package://so_arm100_description/SO-ARM101-Assets/upper_arm_so101_v1.stl" />
         </geometry>
       </collision>
     </link>
     <joint name="${prefix}shoulder_lift_joint" type="revolute">
-      <origin xyz="0 0.1025 0.0306" rpy="0 0 0" />
+      <origin xyz="0 0 0.0624" rpy="3.14159 0 0" />
       <parent link="${prefix}shoulder_link" />
       <child link="${prefix}upper_arm_link" />
-      <axis xyz="1 0 0" />
-      <limit lower="-1.75" upper="1.75" effort="1" velocity="1" />
+      <axis xyz="0 0 1" />
+      <limit effort="10" velocity="10" lower="-1.74533" upper="1.74533" />
     </joint>
     <link name="${prefix}forearm_link">
@@ -166,29 +169,34 @@
         <origin xyz="0 0 0" rpy="0 0 0" />
         <geometry>
-          <mesh
-            filename="package://so_arm100_description/meshes/Lower_Arm.STL"
-          />
-        </geometry>
-        <material name="">
-          <color
-            rgba="0.792156862745098 0.819607843137255 0.933333333333333 1"
-          />
-        </material>
-      </visual>
-      <collision>
-        <origin xyz="0 0 0" rpy="0 0 0" />
-        <geometry>
-          <mesh
-            filename="package://so_arm100_description/meshes/Lower_Arm.STL"
-          />
+          <mesh filename="package://so_arm100_description/SO-ARM101-Assets/under_arm_so101_v1.stl" />
+        </geometry>
+        <material name="3d_printed"/>
+      </visual>
+      <visual>
+        <origin xyz="0 0 0" rpy="0 0 0" />
+        <geometry>
+          <mesh filename="package://so_arm100_description/SO-ARM101-Assets/motor_holder_so101_wrist_v1.stl" />
+        </geometry>
+      </visual>
+      <visual>
+        <origin xyz="0 0 0" rpy="0 0 0" />
+        <geometry>
+          <mesh filename="package://so_arm100_description/SO-ARM101-Assets/sts3215_03a_v1.stl" />
+        </geometry>
+        <material name="sts3215"/>
+      </visual>
+      <collision>
+        <origin xyz="0 0 0" rpy="0 0 0" />
+        <geometry>
+          <mesh filename="package://so_arm100_description/SO-ARM101-Assets/under_arm_so101_v1.stl" />
         </geometry>
       </collision>
     </link>
     <joint name="${prefix}elbow_joint" type="revolute">
-      <origin xyz="0 0.11257 0.028" rpy="0 0 0" />
+      <origin xyz="-0.0303992 -0.0182778 -0.0542" rpy="-1.5708 -1.5708 0" />
       <parent link="${prefix}upper_arm_link" />
       <child link="${prefix}forearm_link" />
-      <axis xyz="1 0 0" />
-      <limit lower="-1.75" upper="1.57" effort="1" velocity="1" />
+      <axis xyz="0 0 1" />
+      <limit effort="10" velocity="10" lower="-1.69" upper="1.69" />
     </joint>
     <link name="${prefix}wrist_1_link">
@@ -211,29 +219,27 @@
         <origin xyz="0 0 0" rpy="0 0 0" />
         <geometry>
-          <mesh
-            filename="package://so_arm100_description/meshes/Wrist_Pitch_Roll.STL"
-          />
-        </geometry>
-        <material name="">
-          <color
-            rgba="0.792156862745098 0.819607843137255 0.933333333333333 1"
-          />
-        </material>
-      </visual>
-      <collision>
-        <origin xyz="0 0 0" rpy="0 0 0" />
-        <geometry>
-          <mesh
-            filename="package://so_arm100_description/meshes/Wrist_Pitch_Roll.STL"
-          />
+          <mesh filename="package://so_arm100_description/SO-ARM101-Assets/sts3215_03a_no_horn_v1.stl" />
+        </geometry>
+        <material name="sts3215"/>
+      </visual>
+      <visual>
+        <origin xyz="0 0 0" rpy="0 0 0" />
+        <geometry>
+          <mesh filename="package://so_arm100_description/SO-ARM101-Assets/wrist_roll_pitch_so101_v2.stl" />
+        </geometry>
+      </visual>
+      <collision>
+        <origin xyz="0 0 0" rpy="0 0 0" />
+        <geometry>
+          <mesh filename="package://so_arm100_description/SO-ARM101-Assets/sts3215_03a_no_horn_v1.stl" />
         </geometry>
       </collision>
     </link>
     <joint name="${prefix}wrist_pitch_joint" type="revolute">
-      <origin xyz="0 0.0052 0.1349" rpy="0 0 0" />
+      <origin xyz="-0.1224 0.0052 0.0187" rpy="-3.14159 0 -3.14159" />
       <parent link="${prefix}forearm_link" />
       <child link="${prefix}wrist_1_link" />
-      <axis xyz="1 0 0" />
-      <limit lower="-3.5" upper="0.2" effort="1" velocity="1" />
+      <axis xyz="0 0 1" />
+      <limit effort="10" velocity="10" lower="-1.65806" upper="1.65806" />
     </joint>
     <link name="${prefix}wrist_2_link">
@@ -256,29 +262,27 @@
         <origin xyz="0 0 0" rpy="0 0 0" />
         <geometry>
-          <mesh
-            filename="package://so_arm100_description/meshes/Fixed_Jaw.STL"
-          />
-        </geometry>
-        <material name="">
-          <color
-            rgba="0.792156862745098 0.819607843137255 0.933333333333333 1"
-          />
-        </material>
-      </visual>
-      <collision>
-        <origin xyz="0 0 0" rpy="0 0 0" />
-        <geometry>
-          <mesh
-            filename="package://so_arm100_description/meshes/Fixed_Jaw.STL"
-          />
+          <mesh filename="package://so_arm100_description/SO-ARM101-Assets/sts3215_03a_v1.stl" />
+        </geometry>
+        <material name="sts3215"/>
+      </visual>
+      <visual>
+        <origin xyz="0 0 0" rpy="0 0 0" />
+        <geometry>
+          <mesh filename="package://so_arm100_description/SO-ARM101-Assets/wrist_roll_follower_so101_v1.stl" />
+        </geometry>
+      </visual>
+      <collision>
+        <origin xyz="0 0 0" rpy="0 0 0" />
+        <geometry>
+          <mesh filename="package://so_arm100_description/SO-ARM101-Assets/sts3215_03a_v1.stl" />
         </geometry>
       </collision>
     </link>
     <joint name="${prefix}wrist_roll_joint" type="revolute">
-      <origin xyz="0 -0.0601 0" rpy="0 0 0" />
+      <origin xyz="5.55112e-17 -0.0611 0.0181" rpy="1.5708 0.0486795 3.14159" />
       <parent link="${prefix}wrist_1_link" />
       <child link="${prefix}wrist_2_link" />
-      <axis xyz="0 1 0" />
-      <limit lower="-1.0" upper="4.0" effort="1" velocity="1" />
+      <axis xyz="0 0 1" />
+      <limit effort="10" velocity="10" lower="-2.74385" upper="2.84121" />
     </joint>
     <link name="${prefix}jaw_link">
@@ -301,29 +305,35 @@
         <origin xyz="0 0 0" rpy="0 0 0" />
         <geometry>
-          <mesh
-            filename="package://so_arm100_description/meshes/Moving_Jaw.STL"
-          />
-        </geometry>
-        <material name="">
-          <color
-            rgba="0.792156862745098 0.819607843137255 0.933333333333333 1"
-          />
-        </material>
-      </visual>
-      <collision>
-        <origin xyz="0 0 0" rpy="0 0 0" />
-        <geometry>
-          <mesh
-            filename="package://so_arm100_description/meshes/Moving_Jaw.STL"
-          />
-        </geometry>
-      </collision>
-    </link>
+          <mesh filename="package://so_arm100_description/SO-ARM101-Assets/moving_jaw_so101_v1.stl" />
+        </geometry>
+        <material name="3d_printed"/>
+      </visual>
+      <collision>
+        <origin xyz="0 0 0" rpy="0 0 0" />
+        <geometry>
+          <mesh filename="package://so_arm100_description/SO-ARM101-Assets/moving_jaw_so101_v1.stl" />
+        </geometry>
+      </collision>
+    </link>
+    <!-- Gripper frame (dummy link + fixed joint) -->
+    <link name="${prefix}gripper_frame_link">
+      <inertial>
+        <origin xyz="0 0 0" rpy="0 0 0"/>
+        <mass value="1e-9"/>
+        <inertia ixx="0" ixy="0" ixz="0" iyy="0" iyz="0" izz="0"/>
+      </inertial>
+    </link>
+    <joint name="${prefix}gripper_frame_joint" type="fixed">
+      <origin xyz="-0.0079 -0.000218121 -0.0981274" rpy="0 3.14159 0"/>
+      <parent link="${prefix}wrist_2_link"/>
+      <child link="${prefix}gripper_frame_link"/>
+      <axis xyz="0 0 0"/>
+    </joint>
     <joint name="${prefix}jaw_joint" type="revolute">
-      <origin xyz="-0.0202 -0.0244 0" rpy="3.1416 0 3.1416" />
+      <origin xyz="0.0202 0.0188 -0.0234" rpy="1.5708 -5.24284e-08 -1.41553e-15"/>
       <parent link="${prefix}wrist_2_link" />
       <child link="${prefix}jaw_link" />
       <axis xyz="0 0 1" />
-      <limit lower="-0.22" upper="2.0" effort="1" velocity="1" />
+      <limit effort="10" velocity="10" lower="-0.174533" upper="1.74533" />
     </joint>
   </xacro:macro>
