Commit message: updated the  file path for mesh files

File: so_arm100_description/SO-ARM101-Assets/so101_new_calib.urdf (robot description, URDF)
Before this commit: robot so101_new_calib, 8 links, 7 joints
Links:
- link base_link: geometry collision mesh filename=package://so_arm100_description/SO-ARM101-Assets/base_motor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; collision mesh filename=package://so_arm100_description/SO-ARM101-Assets/base_so101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
- link gripper_link: geometry collision mesh filename=package://so_arm100_description/SO-ARM101-Assets/sts3215_03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; collision mesh filename=package://so_arm100_description/SO-ARM101-Assets/wrist_roll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
- link lower_arm_link: geometry collision mesh filename=package://so_arm100_description/SO-ARM101-Assets/motor_hold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; collision mesh filename=package://so_arm100_description/SO-ARM101-Assets/sts3215_03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
- link moving_jaw_so101_v1_link: geometry collision mesh filename=package://so_arm100_description/SO-ARM101-Assets/moving_jaw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; visual mesh filename=package://so_arm100_description/SO-ARM101-Assets/moving_jaw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
- link shoulder_link: geometry collision mesh filename=package://so_arm100_description/SO-ARM101-Assets/motor_hold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; collision mesh filename=package://so_arm100_description/SO-ARM101-Assets/rotation_p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
- link upper_arm_link: geometry collision mesh filename=package://so_arm100_description/SO-ARM101-Assets/sts3215_03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; collision mesh filename=package://so_arm100_description/SO-ARM101-Assets/upper_arm_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
- link wrist_link: geometry collision mesh filename=package://so_arm100_description/SO-ARM101-Assets/sts3215_03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; collision mesh filename=package://so_arm100_description/SO-ARM101-Assets/wrist_roll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
