Commit message: With this update, the robot body parts appear as connected in RViz. However, the visualized and the physical robot have clearly different joint state

File: so_arm100_description/urdf/so_arm100_macro.xacro (robot description, xacro)
@@ -1,75 +1,75 @@
-<?xml version="1.0" encoding="utf-8" ?>
-<!-- Copied from
-SO-ARM100/URDF/SO_5DOF_ARM100_8j_URDF.SLDASM/urdf/SO_5DOF_ARM100_8j_URDF.SLDASM.urdf with minimal
-changes:
-- package://SO_5DOF_ARM100_8j_URDF.SLDASM -> package://so_arm100_description
-- Moving Jaw.STL -> Moving_Jaw.STL
-- Link names:
-  - Base -> base
-  - Rotation_Pitch -> shoulder_link
-  - Upper_Arm -> upper_arm_link
-  - Lower_Arm -> forearm_link
-  - Wrist_Pitch_Roll -> wrist_1_link
-  - Fixed_Jaw -> wrist_2_link
-  - Moving Jaw -> jaw_link
-- Joint names:
-  - Rotation -> shoulder_pan_joint
-  - Pitch -> shoulder_lift_joint
-  - Elbow -> elbow_joint
-  - Wrist_Pitch -> wrist_pitch_joint
-  - Wrist_Roll -> wrist_roll_joint
-  - Jaw -> jaw_joint
--->
-<robot xmlns:xacro="http://ros.org/wiki/xacro">
+<?xml version="1.0"?>
+<robot xmlns:xacro="http://www.ros.org/wiki/xacro">
+  <material name="3d_printed">
+    <color rgba="1.0 0.82 0.12 1.0" />
+  </material>
+  <material name="sts3215">
+    <color rgba="0.1 0.1 0.1 1.0" />
+  </material>
   <xacro:macro name="so_arm100" params="prefix">
     <link name="${prefix}base">
       <inertial>
-        <origin
-          xyz="-2.45960666746703E-07 0.0311418169687909 0.0175746661003382"
-          rpy="0 0 0"
-        />
-        <mass value="0.193184127927598" />
-        <inertia
-          ixx="0.000137030709467877"
-          ixy="2.10136126944992E-08"
-          ixz="4.24087422551286E-09"
-          iyy="0.000169089551209259"
-          iyz="2.26514711036514E-05"
-          izz="0.000145097720857224"
-        />
-      </inertial>
-      <visual>
-        <origin xyz="0 0 0" rpy="0 0 0" />
+        <origin xyz="0.020739 0.00204287 0.065966" rpy="0 0 0" />
+        <mass value="0.147" />
+        <inertia ixx="0.000136117" ixy="4.59787e-07" ixz="9.75275e-08" iyy="0.000114686" iyz="-4.97151e-06" izz="0.000130364" />
+      </inertial>
+      <visual>
+        <origin xyz="0.0206915 0.0221255 0.0300817" rpy="1.5708 -1.23909e-16 2.33147e-15" />
         <geometry>
           <mesh filename="package://so_arm100_description/SO-ARM101-Assets/base_motor_holder_so101_v1.stl" />
         </geometry>
-        <material name="">
-          <color
-            rgba="0.792156862745098 0.819607843137255 0.933333333333333 1"
-          />
-        </material>
-      </visual>
-      <collision>
-        <origin xyz="0 0 0" rpy="0 0 0" />
+        <material name="3d_printed" />
+      </visual>
+      <collision>
+        <origin xyz="0.0206915 0.0221255 0.0300817" rpy="1.5708 -1.23909e-16 2.33147e-15" />
         <geometry>
           <mesh filename="package://so_arm100_description/SO-ARM101-Assets/base_motor_holder_so101_v1.stl" />
         </geometry>
       </collision>
+      <visual>
+        <origin xyz="0.0207909 0.0221255 0.0300817" rpy="1.5708 -0 0" />
+        <geometry>
+          <mesh filename="package://so_arm100_description/SO-ARM101-Assets/base_so101_v2.stl" />
+        </geometry>
+        <material name="3d_printed" />
+      </visual>
+      <collision>
+        <origin xyz="0.0207909 0.0221255 0.0300817" rpy="1.5708 -0 0" />
+        <geometry>
+          <mesh filename="package://so_arm100_description/SO-ARM101-Assets/base_so101_v2.stl" />
+        </geometry>
+      </collision>
+      <visual>
+        <origin xyz="0.0207909 -0.0105745 0.0761817" rpy="-2.20282e-15 2.77556e-17 -1.5708" />
+        <geometry>
+          <mesh filename="package://so_arm100_description/SO-ARM101-Assets/sts3215_03a_v1.stl" />
+        </geometry>
+        <material name="sts3215" />
+      </visual>
+      <collision>
+        <origin xyz="0.0207909 -0.0105745 0.0761817" rpy="-2.20282e-15 2.77556e-17 -1.5708" />
+        <geometry>
+          <mesh filename="package://so_arm100_description/SO-ARM101-Assets/sts3215_03a_v1.stl" />
+        </geometry>
+      </collision>
+      <visual>
+        <origin xyz="0.0205915 0.0467435 0.0798817" rpy="1.5708 -1.21716e-14 2.33147e-15" />
+        <geometry>
+          <mesh filename="package://so_arm100_description/SO-ARM101-Assets/waveshare_mounting_plate_so101_v2.stl" />
+        </geometry>
+        <material name="3d_printed" />
+      </visual>
+      <collision>
+        <origin xyz="0.0205915 0.0467435 0.0798817" rpy="1.5708 -1.21716e-14 2.33147e-15" />
+        <geometry>
+          <mesh filename="package://so_arm100_description/SO-ARM101-Assets/waveshare_mounting_plate_so101_v2.stl" />
+        </geometry>
+      </collision>
     </link>
     <link name="${prefix}shoulder_link">
       <inertial>
-        <origin
-          xyz="-9.07886224712597E-05 0.0590971820568318 0.031089016892169"
-          rpy="0 0 0"
-        />
-        <mass value="0.119226314127197" />
-        <inertia
-          ixx="5.90408775624429E-05"
-          ixy="4.90800532852998E-07"
-          ixz="-5.90451772654387E-08"
-          iyy="3.21498601038881E-05"
-          iyz="-4.58026206663885E-06"
-          izz="5.86058514263952E-05"
-        />
+        <origin xyz="-0.0307604 -1.66727e-05 -0.0252713" rpy="0 0 0" />
+        <mass value="0.100006" />
+        <inertia ixx="8.3759e-05" ixy="7.55525e-08" ixz="-1.16342e-06" iyy="8.10403e-05" iyz="1.54663e-07" izz="2.39783e-05" />
       </inertial>
       <visual>
@@ -78,6 +78,12 @@
           <mesh filename="package://so_arm100_description/SO-ARM101-Assets/sts3215_03a_v1.stl" />
         </geometry>
-        <material name="sts3215"/>
-      </visual>
+        <material name="sts3215" />
+      </visual>
+      <collision>
+        <origin xyz="-0.0303992 0.000422241 -0.0417" rpy="1.5708 1.5708 0" />
+        <geometry>
+          <mesh filename="package://so_arm100_description/SO-ARM101-Assets/sts3215_03a_v1.stl" />
+        </geometry>
+      </collision>
       <visual>
         <origin xyz="-0.0675992 -0.000177759 0.0158499" rpy="1.5708 -1.5708 0" />
@@ -85,57 +91,61 @@
           <mesh filename="package://so_arm100_description/SO-ARM101-Assets/motor_holder_so101_base_v1.stl" />
         </geometry>
-        <material name="3d_printed"/>
-      </visual>
-      <visual>
-        <origin xyz="0 0 0" rpy="0 0 0" />
+        <material name="3d_printed" />
+      </visual>
+      <collision>
+        <origin xyz="-0.0675992 -0.000177759 0.0158499" rpy="1.5708 -1.5708 0" />
+        <geometry>
+          <mesh filename="package://so_arm100_description/SO-ARM101-Assets/motor_holder_so101_base_v1.stl" />
+        </geometry>
+      </collision>
+      <visual>
+        <origin xyz="0.0122008 2.22413e-05 0.0464" rpy="-1.5708 -0 0" />
         <geometry>
           <mesh filename="package://so_arm100_description/SO-ARM101-Assets/rotation_pitch_so101_v1.stl" />
         </geometry>
-      </visual>
-      <collision>
-        <origin xyz="-0.0303992 0.000422241 -0.0417" rpy="1.5708 1.5708 0" />
-        <geometry>
-          <mesh filename="package://so_arm100_description/SO-ARM101-Assets/sts3215_03a_v1.stl" />
+        <material name="3d_printed" />
+      </visual>
+      <collision>
+        <origin xyz="0.0122008 2.22413e-05 0.0464" rpy="-1.5708 -0 0" />
+        <geometry>
+          <mesh filename="package://so_arm100_description/SO-ARM101-Assets/rotation_pitch_so101_v1.stl" />
         </geometry>
       </collision>
     </link>
     <joint name="${prefix}shoulder_pan_joint" type="revolute">
-      <origin xyz="0.0388353 0 0.0459" rpy="0 0 0" />
+      <origin xyz="0.0388353 -8.97657e-09 0.0624" rpy="3.14159 4.18253e-17 -3.14159" />
       <parent link="${prefix}base" />
       <child link="${prefix}shoulder_link" />
       <axis xyz="0 0 1" />
-      <limit effort="10" velocity="10" lower="-1.91986" upper="1.91986" />
+      <limit lower="-1.91986" upper="1.91986" effort="10" velocity="10" />
     </joint>
     <link name="${prefix}upper_arm_link">
       <inertial>
-        <origin
-          xyz="-1.7205170190925E-05 0.0701802156327694 0.00310545118155671"
-          rpy="0 0 0"
-        />
-        <mass value="0.162409284599177" />
-        <inertia
-          ixx="0.000167153146617081"
-          ixy="1.03902689187701E-06"
-          ixz="-1.20161820645189E-08"
-          iyy="7.01946992214245E-05"
-          iyz="2.11884806298698E-06"
-          izz="0.000213280241160769"
-        />
-      </inertial>
-      <visual>
-        <origin xyz="0 0 0" rpy="0 0 0" />
-        <geometry>
-          <mesh filename="package://so_arm100_description/SO-ARM101-Assets/sts3215_03a_v1.stl" />
-        </geometry>
-        <material name="sts3215"/>
-      </visual>
-      <visual>
-        <origin xyz="0 0 0" rpy="0 0 0" />
+        <origin xyz="-0.0898471 -0.00838224 0.0184089" rpy="0 0 0" />
+        <mass value="0.103" />
+        <inertia ixx="4.08002e-05" ixy="-1.97819e-05" ixz="-4.03016e-08" iyy="0.000147318" iyz="8.97326e-09" izz="0.000142487" />
+      </inertial>
+      <visual>
+        <origin xyz="-0.11257 -0.0155 0.0187" rpy="-3.14159 -6.8695e-16 -1.5708" />
+        <geometry>
+          <mesh filename="package://so_arm100_description/SO-ARM101-Assets/sts3215_03a_v1.stl" />
+        </geometry>
+        <material name="sts3215" />
+      </visual>
+      <collision>
+        <origin xyz="-0.11257 -0.0155 0.0187" rpy="-3.14159 -6.8695e-16 -1.5708" />
+        <geometry>
+          <mesh filename="package://so_arm100_description/SO-ARM101-Assets/sts3215_03a_v1.stl" />
+        </geometry>
+      </collision>
+      <visual>
+        <origin xyz="-0.065085 0.012 0.0182" rpy="3.14159 -9.35612e-32 0" />
         <geometry>
           <mesh filename="package://so_arm100_description/SO-ARM101-Assets/upper_arm_so101_v1.stl" />
         </geometry>
-      </visual>
-      <collision>
-        <origin xyz="0 0 0" rpy="0 0 0" />
+        <material name="3d_printed" />
+      </visual>
+      <collision>
+        <origin xyz="-0.065085 0.012 0.0182" rpy="3.14159 -9.35612e-32 0" />
         <geometry>
           <mesh filename="package://so_arm100_description/SO-ARM101-Assets/upper_arm_so101_v1.stl" />
@@ -144,136 +154,133 @@
     </link>
     <joint name="${prefix}shoulder_lift_joint" type="revolute">
-      <origin xyz="0 0 0.0624" rpy="3.14159 0 0" />
+      <origin xyz="-0.0303992 -0.0182778 -0.0542" rpy="-1.5708 -1.5708 0" />
       <parent link="${prefix}shoulder_link" />
       <child link="${prefix}upper_arm_link" />
       <axis xyz="0 0 1" />
-      <limit effort="10" velocity="10" lower="-1.74533" upper="1.74533" />
+      <limit lower="-1.74533" upper="1.74533" effort="10" velocity="10" />
     </joint>
     <link name="${prefix}forearm_link">
       <inertial>
-        <origin
-          xyz="-0.00339603710186651 0.00137796353960074 0.0768006751156044"
-          rpy="0 0 0"
-        />
-        <mass value="0.147967774582291" />
-        <inertia
-          ixx="0.000105333995841409"
-          ixy="1.73059237226499E-07"
-          ixz="-1.1720305455211E-05"
-          iyy="0.000138766654485212"
-          iyz="1.77429964684103E-06"
-          izz="5.08741652515214E-05"
-        />
-      </inertial>
-      <visual>
-        <origin xyz="0 0 0" rpy="0 0 0" />
+        <origin xyz="-0.0980701 0.00324376 0.0182831" rpy="0 0 0" />
+        <mass value="0.104" />
+        <inertia ixx="2.87438e-05" ixy="7.41152e-06" ixz="1.26409e-06" iyy="0.000159844" iyz="-4.90188e-08" izz="0.00014529" />
+      </inertial>
+      <visual>
+        <origin xyz="-0.0648499 -0.032 0.0182" rpy="-3.14159 -0 3.9443e-31" />
         <geometry>
           <mesh filename="package://so_arm100_description/SO-ARM101-Assets/under_arm_so101_v1.stl" />
         </geometry>
-        <material name="3d_printed"/>
-      </visual>
-      <visual>
-        <origin xyz="0 0 0" rpy="0 0 0" />
+        <material name="3d_printed" />
+      </visual>
+      <collision>
+        <origin xyz="-0.0648499 -0.032 0.0182" rpy="-3.14159 -0 3.9443e-31" />
+        <geometry>
+          <mesh filename="package://so_arm100_description/SO-ARM101-Assets/under_arm_so101_v1.stl" />
+        </geometry>
+      </collision>
+      <visual>
+        <origin xyz="-0.0648499 -0.032 0.018" rpy="-3.14159 4.73317e-30 7.88861e-31" />
         <geometry>
           <mesh filename="package://so_arm100_description/SO-ARM101-Assets/motor_holder_so101_wrist_v1.stl" />
         </geometry>
-      </visual>
-      <visual>
-        <origin xyz="0 0 0" rpy="0 0 0" />
-        <geometry>
-          <mesh filename="package://so_arm100_description/SO-ARM101-Assets/sts3215_03a_v1.stl" />
-        </geometry>
-        <material name="sts3215"/>
-      </visual>
-      <collision>
-        <origin xyz="0 0 0" rpy="0 0 0" />
-        <geometry>
-          <mesh filename="package://so_arm100_description/SO-ARM101-Assets/under_arm_so101_v1.stl" />
+        <material name="3d_printed" />
+      </visual>
+      <collision>
+        <origin xyz="-0.0648499 -0.032 0.018" rpy="-3.14159 4.73317e-30 7.88861e-31" />
+        <geometry>
+          <mesh filename="package://so_arm100_description/SO-ARM101-Assets/motor_holder_so101_wrist_v1.stl" />
+        </geometry>
+      </collision>
+      <visual>
+        <origin xyz="-0.1224 0.0052 0.0187" rpy="-3.14159 -3.58047e-15 -3.14159" />
+        <geometry>
+          <mesh filename="package://so_arm100_description/SO-ARM101-Assets/sts3215_03a_v1.stl" />
+        </geometry>
+        <material name="sts3215" />
+      </visual>
+      <collision>
+        <origin xyz="-0.1224 0.0052 0.0187" rpy="-3.14159 -3.58047e-15 -3.14159" />
+        <geometry>
+          <mesh filename="package://so_arm100_description/SO-ARM101-Assets/sts3215_03a_v1.stl" />
         </geometry>
       </collision>
     </link>
     <joint name="${prefix}elbow_joint" type="revolute">
-      <origin xyz="-0.0303992 -0.0182778 -0.0542" rpy="-1.5708 -1.5708 0" />
+      <origin xyz="-0.11257 -0.028 1.73763e-16" rpy="-3.63608e-16 8.74301e-16 1.5708" />
       <parent link="${prefix}upper_arm_link" />
       <child link="${prefix}forearm_link" />
       <axis xyz="0 0 1" />
-      <limit effort="10" velocity="10" lower="-1.69" upper="1.69" />
+      <limit lower="-1.69" upper="1.69" effort="10" velocity="10" />
     </joint>
     <link name="${prefix}wrist_1_link">
       <inertial>
-        <origin
-          xyz="-0.00852653127372418 -0.0352278997897927 -2.34622481569413E-05"
-          rpy="0 0 0"
-        />
-        <mass value="0.066132067097723" />
-        <inertia
-          ixx="1.95717492443445E-05"
-          ixy="-6.62714374412293E-07"
-          ixz="5.20089016442066E-09"
-          iyy="2.38028417569933E-05"
-          iyz="4.09549055863776E-08"
-          izz="3.4540143384536E-05"
-        />
-      </inertial>
-      <visual>
-        <origin xyz="0 0 0" rpy="0 0 0" />
+        <origin xyz="-0.000103312 -0.0386143 0.0281156" rpy="0 0 0" />
+        <mass value="0.079" />
+        <inertia ixx="3.68263e-05" ixy="1.7893e-08" ixz="-5.28128e-08" iyy="2.5391e-05" iyz="3.6412e-06" izz="2.1e-05" />
+      </inertial>
+      <visual>
+        <origin xyz="5.55112e-17 -0.0424 0.0306" rpy="1.5708 1.5708 0" />
         <geometry>
           <mesh filename="package://so_arm100_description/SO-ARM101-Assets/sts3215_03a_no_horn_v1.stl" />
         </geometry>
-        <material name="sts3215"/>
-      </visual>
-      <visual>
-        <origin xyz="0 0 0" rpy="0 0 0" />
+        <material name="sts3215" />
+      </visual>
+      <collision>
+        <origin xyz="5.55112e-17 -0.0424 0.0306" rpy="1.5708 1.5708 0" />
+        <geometry>
+          <mesh filename="package://so_arm100_description/SO-ARM101-Assets/sts3215_03a_no_horn_v1.stl" />
+        </geometry>
+      </collision>
+      <visual>
+        <origin xyz="0 -0.028 0.0181" rpy="-1.5708 -1.5708 0" />
         <geometry>
           <mesh filename="package://so_arm100_description/SO-ARM101-Assets/wrist_roll_pitch_so101_v2.stl" />
         </geometry>
-      </visual>
-      <collision>
-        <origin xyz="0 0 0" rpy="0 0 0" />
-        <geometry>
-          <mesh filename="package://so_arm100_description/SO-ARM101-Assets/sts3215_03a_no_horn_v1.stl" />
+        <material name="3d_printed" />
+      </visual>
+      <collision>
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
Commit message: correct the origin for base link

File: so_arm100_description/urdf/so_arm100_macro.xacro (robot description, xacro)
@@ -10,7 +10,7 @@
     <link name="${prefix}base">
       <inertial>
-        <origin xyz="0.020739 0.00204287 0.065966" rpy="0 0 0" />
+        <origin xyz="0.0137179 -5.19711e-05 0.0334843" rpy="0 0 0" />
         <mass value="0.147" />
-        <inertia ixx="0.000136117" ixy="4.59787e-07" ixz="9.75275e-08" iyy="0.000114686" iyz="-4.97151e-06" izz="0.000130364" />
+        <inertia ixx="0.000114686" ixy="-4.59787e-07" ixz="4.97151e-06" iyy="0.000136117" iyz="9.75275e-08" izz="0.000130364" />
       </inertial>
       <visual>

Commit message: correct errors for base link by syncing to so101_new_calib.urdf

File: so_arm100_description/urdf/so_arm100_macro.xacro (robot description, xacro)
@@ -15,5 +15,5 @@
       </inertial>
       <visual>
-        <origin xyz="0.0206915 0.0221255 0.0300817" rpy="1.5708 -1.23909e-16 2.33147e-15" />
+        <origin xyz="-0.00636471 -9.94414e-05 -0.0024" rpy="1.5708 -1.67685e-15 1.5708" />
         <geometry>
           <mesh filename="package://so_arm100_description/SO-ARM101-Assets/base_motor_holder_so101_v1.stl" />
@@ -22,5 +22,5 @@
       </visual>
       <collision>
-        <origin xyz="0.0206915 0.0221255 0.0300817" rpy="1.5708 -1.23909e-16 2.33147e-15" />
+        <origin xyz="-0.00636471 -9.94414e-05 -0.0024" rpy="1.5708 -1.67685e-15 1.5708" />
         <geometry>
           <mesh filename="package://so_arm100_description/SO-ARM101-Assets/base_motor_holder_so101_v1.stl" />
@@ -28,5 +28,5 @@
       </collision>
       <visual>
-        <origin xyz="0.0207909 0.0221255 0.0300817" rpy="1.5708 -0 0" />
+        <origin xyz="-0.00636471 -8.97657e-09 -0.0024" rpy="1.5708 -2.78073e-29 1.5708" />
         <geometry>
           <mesh filename="package://so_arm100_description/SO-ARM101-Assets/base_so101_v2.stl" />
@@ -35,5 +35,5 @@
       </visual>
       <collision>
-        <origin xyz="0.0207909 0.0221255 0.0300817" rpy="1.5708 -0 0" />
+        <origin xyz="-0.00636471 -8.97657e-09 -0.0024" rpy="1.5708 -2.78073e-29 1.5708" />
         <geometry>
           <mesh filename="package://so_arm100_description/SO-ARM101-Assets/base_so101_v2.stl" />
@@ -41,18 +41,18 @@
       </collision>
       <visual>
-        <origin xyz="0.0207909 -0.0105745 0.0761817" rpy="-2.20282e-15 2.77556e-17 -1.5708" />
-        <geometry>
-          <mesh filename="package://so_arm100_description/SO-ARM101-Assets/sts3215_03a_v1.stl" />
-        </geometry>
-        <material name="sts3215" />
-      </visual>
-      <collision>
-        <origin xyz="0.0207909 -0.0105745 0.0761817" rpy="-2.20282e-15 2.77556e-17 -1.5708" />
-        <geometry>
-          <mesh filename="package://so_arm100_description/SO-ARM101-Assets/sts3215_03a_v1.stl" />
-        </geometry>
-      </collision>
-      <visual>
-        <origin xyz="0.0205915 0.0467435 0.0798817" rpy="1.5708 -1.21716e-14 2.33147e-15" />
+        <origin xyz="0.0263353 -8.97657e-09 0.0437" rpy="-8.21148e-16 7.84513e-18 1.249e-15" />
+        <geometry>
+          <mesh filename="package://so_arm100_description/SO-ARM101-Assets/sts3215_03a_v1.stl" />
+        </geometry>
+        <material name="sts3215" />
+      </visual>
+      <collision>
+        <origin xyz="0.0263353 -8.97657e-09 0.0437" rpy="-8.21148e-16 7.84513e-18 1.249e-15" />
+        <geometry>
+          <mesh filename="package://so_arm100_description/SO-ARM101-Assets/sts3215_03a_v1.stl" />
+        </geometry>
+      </collision>
+      <visual>
+        <origin xyz="-0.0309827 -0.000199441 0.0474" rpy="1.5708 -1.35493e-14 1.5708" />
         <geometry>
           <mesh filename="package://so_arm100_description/SO-ARM101-Assets/waveshare_mounting_plate_so101_v2.stl" />
@@ -61,5 +61,5 @@
       </visual>
       <collision>
-        <origin xyz="0.0205915 0.0467435 0.0798817" rpy="1.5708 -1.21716e-14 2.33147e-15" />
+        <origin xyz="-0.0309827 -0.000199441 0.0474" rpy="1.5708 -1.35493e-14 1.5708" />
         <geometry>
           <mesh filename="package://so_arm100_description/SO-ARM101-Assets/waveshare_mounting_plate_so101_v2.stl" />
